Commit message: add friction simulation

File: robot_gazebo/urdf/pav_s01/macros.xacro (robot description, xacro)
@@ -26,3 +26,13 @@
   </transmission>
 </xacro:macro>
+<xacro:macro name="wheel_friction" params="name">
+  <surface>
+      <friction>
+        <ode>
+            <mu>999999999999999999</mu>
+            <mu2>999999999999999999</mu2>
+        </ode>
+      </friction>
+  </surface>
+</xacro:macro>
 </robot>

File: robot_gazebo/urdf/pav_s01/pav_s01.xacro (robot description, xacro)
@@ -1,4 +1,7 @@
 <?xml version="1.0" encoding="utf-8"?>
 <robot name="$(arg robot_name)" xmlns:xacro="http://ros.org/wiki/xacro">
+  <xacro:property name="M_PI" value="3.141592653589793" />
+  <xacro:property name="rotation_fiction" value="1"/>
+  <xacro:property name="mu" value="9999999999.0"/>
   <xacro:include filename="$(find robot_gazebo)/urdf/pav_s01/macros.xacro" />
   <link name="$(arg robot_name)/base_footprint"/>
@@ -36,5 +39,5 @@
   <link name="$(arg robot_name)/shell_link">
     <visual>
-      <origin xyz="0 0 0" rpy="1.57 0 -1.57" />
+      <origin xyz="0 0 0" rpy="${M_PI/2} 0 -${M_PI/2}" />
       <geometry>
         <mesh filename="package://robot_gazebo/models/robots/pav_s01/shell_pav_s01.STL" scale="0.001 0.001 0.001"/>
@@ -58,5 +61,5 @@
         <mesh filename="package://robot_gazebo/models/robots/pav_s01/wheel_link.STL" />
       </geometry>
-      <!-- <origin xyz="0 0 0" rpy="1.57 0 0" />
+      <!-- <origin xyz="0 0 0" rpy="${M_PI/2} 0 0" />
       <geometry>
         <cylinder radius="0.035" length="0.02" />
@@ -67,9 +70,10 @@
     </visual>
     <collision>
-      <origin xyz="0 0 0" rpy="1.57 0 0" />
-      <geometry>
-        <cylinder radius="0.035" length="0.02" />
-      </geometry>
-    </collision>
+      <origin xyz="0 0 0" rpy="${M_PI/2} 0 0" />
+      <geometry>
+        <cylinder radius="0.035" length="0.02" />
+      </geometry>
+    </collision>
+    <xacro:wheel_friction name="${mu}" />
   </link>
   <joint name="right_rear_wheel_link_joint" type="continuous">
@@ -79,4 +83,5 @@
     <axis xyz="0 1 0" />
     <limit effort="10" velocity="1000" />
+    <dynamics damping="0.0" friction="${rotation_fiction}"/>
   </joint>
   <xacro:wheel_transmission name="right_rear_wheel_link" />
@@ -88,9 +93,9 @@
     </inertial>
     <visual>
-      <origin xyz="0 0 0" rpy="0 0 3.14" />
+      <origin xyz="0 0 0" rpy="0 0 ${M_PI}" />
       <geometry>
         <mesh filename="package://robot_gazebo/models/robots/pav_s01/wheel_link.STL" />
       </geometry>
-      <!-- <origin xyz="0 0 0" rpy="1.57 0 0" />
+      <!-- <origin xyz="0 0 0" rpy="${M_PI/2} 0 0" />
       <geometry>
         <cylinder radius="0.035" length="0.02" />
@@ -101,9 +106,10 @@
     </visual>
     <collision>
-      <origin xyz="0 0 0" rpy="1.57 0 0" />
-      <geometry>
-        <cylinder radius="0.035" length="0.02" />
-      </geometry>
-    </collision>
+      <origin xyz="0 0 0" rpy="${M_PI/2} 0 0" />
+      <geometry>
+        <cylinder radius="0.035" length="0.02" />
+      </geometry>
+    </collision>
+    <xacro:wheel_friction name="${mu}" />
   </link>
   <joint name="left_rear_wheel_link_joint" type="continuous">
@@ -113,4 +119,5 @@
     <axis xyz="0 1 0" />
     <limit effort="10" velocity="1000" />
+    <dynamics damping="0.0" friction="${rotation_fiction}"/>
   </joint>
   <xacro:wheel_transmission name="left_rear_wheel_link" />
@@ -126,5 +133,5 @@
         <mesh filename="package://robot_gazebo/models/robots/pav_s01/steer_hinge_link.STL" />
       </geometry>
-      <!-- <origin xyz="0.0 0.0 0.0" rpy="1.57 0.0 0.0" />
+      <!-- <origin xyz="0.0 0.0 0.0" rpy="${M_PI/2} 0.0 0.0" />
       <geometry>
           <cylinder radius="0.01" length="0.005" />
@@ -142,5 +149,5 @@
           <cylinder radius="0.01" length="0.005" />
       </geometry>
-      <origin xyz="0.0 0.0 0.0" rpy="1.57 0.0 0.0" />
+      <origin xyz="0.0 0.0 0.0" rpy="${M_PI/2} 0.0 0.0" />
     </collision>
   </link>
@@ -164,5 +171,5 @@
         <mesh filename="package://robot_gazebo/models/robots/pav_s01/steer_hinge_link.STL" />
       </geometry>
-      <!-- <origin xyz="0.0 0.0 0.0" rpy="1.57 0.0 0.0" />
+      <!-- <origin xyz="0.0 0.0 0.0" rpy="${M_PI/2} 0.0 0.0" />
       <geometry>
           <cylinder radius="0.01" length="0.005" />
@@ -182,5 +189,5 @@
             <cylinder radius="0.01" length="0.005" />
         </geometry>
-        <origin xyz="0.0 0.0 0.0" rpy="1.57 0.0 0.0" />
+        <origin xyz="0.0 0.0 0.0" rpy="${M_PI/2} 0.0 0.0" />
       </collision>
   </link>
@@ -204,5 +211,5 @@
         <mesh filename="package://robot_gazebo/models/robots/pav_s01/wheel_link.STL" />
       </geometry>
-      <!-- <origin xyz="0 0 0" rpy="1.57 0 0" />
+      <!-- <origin xyz="0 0 0" rpy="${M_PI/2} 0 0" />
       <geometry>
         <cylinder radius="0.035" length="0.02" />
@@ -213,9 +220,10 @@
     </visual>
     <collision>
-      <origin xyz="0 0 0" rpy="1.57 0 0" />
-      <geometry>
-        <cylinder radius="0.035" length="0.02" />
-      </geometry>
-    </collision>
+      <origin xyz="0 0 0" rpy="${M_PI/2} 0 0" />
+      <geometry>
+        <cylinder radius="0.035" length="0.02" />
+      </geometry>
+    </collision>
+    <xacro:wheel_friction name="${mu}" />
   </link>
   <joint name="right_front_wheel_link_joint" type="continuous">
@@ -225,4 +233,5 @@
     <axis xyz="0 1 0" />
     <limit effort="10" velocity="1000" />
+    <dynamics damping="0.0" friction="${rotation_fiction}"/>
   </joint>
   <xacro:wheel_transmission name="right_front_wheel_link" />
@@ -234,9 +243,9 @@
     </inertial>
     <visual>
-      <origin xyz="0 0 0" rpy="0 0 3.14" />
+      <origin xyz="0 0 0" rpy="0 0 ${M_PI}" />
       <geometry>
         <mesh filename="package://robot_gazebo/models/robots/pav_s01/wheel_link.STL" />
       </geometry>
-      <!-- <origin xyz="0 0 0" rpy="1.57 0 0" />
+      <!-- <origin xyz="0 0 0" rpy="${M_PI/2} 0 0" />
       <geometry>
         <cylinder radius="0.035" length="0.02" />
@@ -247,9 +256,10 @@
     </visual>
     <collision>
-      <origin xyz="0 0 0" rpy="1.57 0 0" />
-      <geometry>
-        <cylinder radius="0.035" length="0.02" />
-      </geometry>
-    </collision>
+      <origin xyz="0 0 0" rpy="${M_PI/2} 0 0" />
+      <geometry>
+        <cylinder radius="0.035" length="0.02" />
+      </geometry>
+    </collision>
+    <xacro:wheel_friction name="${mu}" />
   </link>
   <joint name="left_front_wheel_link_joint" type="continuous">
@@ -259,4 +269,5 @@
     <axis xyz="0 1 0" />
     <limit effort="10" velocity="1000" />
+    <dynamics damping="0.0" friction="${rotation_fiction}"/>
   </joint>
   <xacro:wheel_transmission name="left_front_wheel_link" />
