Commit message: add prefix to links

File: robot_gazebo/urdf/pav_s01/pav_s01.xacro (robot description, xacro)
@@ -2,6 +2,6 @@
 <robot name="$(arg robot_name)" xmlns:xacro="http://ros.org/wiki/xacro">
   <xacro:include filename="$(find robot_gazebo)/urdf/pav_s01/macros.xacro" />
-  <link name="base_footprint"/>
-  <link name="base_link">
+  <link name="$(arg robot_name)/base_footprint"/>
+  <link name="$(arg robot_name)/base_link">
     <inertial>
       <origin xyz="-0.02 0 0" rpy="0 0 0" />
@@ -29,10 +29,10 @@
     </collision>
   </link>
-  <joint name="base_joint" type="fixed">
-    <parent link="base_footprint"/>
-    <child link="base_link"/>
+  <joint name="$(arg robot_name)/base_joint" type="fixed">
+    <parent link="$(arg robot_name)/base_footprint"/>
+    <child link="$(arg robot_name)/base_link"/>
     <origin xyz="0.0 0.0 0.09" rpy="0 0 0"/>
   </joint>
-  <link name="shell_link">
+  <link name="$(arg robot_name)/shell_link">
     <visual>
       <origin xyz="0 0 0" rpy="1.57 0 -1.57" />
@@ -42,10 +42,10 @@
     </visual>
   </link>
-  <joint name="shell_link_joint" type="fixed">
-    <parent link="base_link"/>
-    <child link="shell_link"/>
+  <joint name="$(arg robot_name)/shell_link_joint" type="fixed">
+    <parent link="$(arg robot_name)/base_link"/>
+    <child link="$(arg robot_name)/shell_link"/>
     <origin xyz="-0.02 0.0 -0.085" rpy="0 0 0"/>
   </joint>
-  <link name="right_rear_wheel_link">
+  <link name="$(arg robot_name)/right_rear_wheel_link">
     <inertial>
       <origin xyz="0 0 0 " rpy="0 0 0" />
@@ -74,6 +74,6 @@
   </link>
   <joint name="right_rear_wheel_link_joint" type="continuous">
-    <parent link="base_link" />
-    <child link="right_rear_wheel_link" />
+    <parent link="$(arg robot_name)/base_link" />
+    <child link="$(arg robot_name)/right_rear_wheel_link" />
     <origin xyz="-0.139 -0.09 -0.055" rpy="0 0 0" />
     <axis xyz="0 1 0" />
@@ -81,5 +81,5 @@
   </joint>
   <xacro:wheel_transmission name="right_rear_wheel_link" />
-  <link name="left_rear_wheel_link">
+  <link name="$(arg robot_name)/left_rear_wheel_link">
     <inertial>
       <origin xyz="0 0 0 " rpy="0 0 0" />
@@ -108,6 +108,6 @@
   </link>
   <joint name="left_rear_wheel_link_joint" type="continuous">
-    <parent link="base_link" />
-    <child link="left_rear_wheel_link" />
+    <parent link="$(arg robot_name)/base_link" />
+    <child link="$(arg robot_name)/left_rear_wheel_link" />
     <origin xyz="-0.139 0.09 -0.055" rpy="0 0 0" />
     <axis xyz="0 1 0" />
@@ -115,5 +115,5 @@
   </joint>
   <xacro:wheel_transmission name="left_rear_wheel_link" />
-  <link name="left_front_steer_hinge_link">
+  <link name="$(arg robot_name)/left_front_steer_hinge_link">
     <inertial>
       <origin xyz="0 0 0" rpy="0 0 0" />
@@ -147,11 +147,11 @@
   <joint name="left_front_steer_hinge_link_joint" type="revolute">
     <origin xyz="0.095 0.065 -0.0525" rpy="0 0 0" />
-    <parent link="base_link" />
-    <child link="left_front_steer_hinge_link" />
+    <parent link="$(arg robot_name)/base_link" />
+    <child link="$(arg robot_name)/left_front_steer_hinge_link" />
     <axis xyz="0 0 1" />
     <limit lower="-0.6" upper="0.6" effort="5" velocity="1000" />
   </joint>
   <xacro:steering_hinge_transmission name="left_front_steer_hinge_link" />
-  <link name="right_front_steer_hinge_link">
+  <link name="$(arg robot_name)/right_front_steer_hinge_link">
     <inertial>
       <origin xyz="0 0 0" rpy="0 0 0" />
@@ -186,6 +186,6 @@
   </link>
   <joint name="right_front_steer_hinge_link_joint" type="revolute">
-    <parent link="base_link" />
-    <child link="right_front_steer_hinge_link" />
+    <parent link="$(arg robot_name)/base_link" />
+    <child link="$(arg robot_name)/right_front_steer_hinge_link" />
     <origin xyz="0.095 -0.065 -0.0525" rpy="0 0 0" />
     <axis xyz="0 0 1" />
@@ -193,5 +193,5 @@
   </joint>
   <xacro:steering_hinge_transmission name="right_front_steer_hinge_link" />
-  <link name="right_front_wheel_link">
+  <link name="$(arg robot_name)/right_front_wheel_link">
     <inertial>
       <origin xyz="0 0 0 " rpy="0 0 0" />
@@ -220,6 +220,6 @@
   </link>
   <joint name="right_front_wheel_link_joint" type="continuous">
-    <parent link="right_front_steer_hinge_link" />
-    <child link="right_front_wheel_link" />
+    <parent link="$(arg robot_name)/right_front_steer_hinge_link" />
+    <child link="$(arg robot_name)/right_front_wheel_link" />
     <origin xyz="0 -0.025 0" rpy="0 0 0" />
     <axis xyz="0 1 0" />
@@ -227,5 +227,5 @@
   </joint>
   <xacro:wheel_transmission name="right_front_wheel_link" />
-  <link name="left_front_wheel_link">
+  <link name="$(arg robot_name)/left_front_wheel_link">
     <inertial>
       <origin xyz="0 0 0 " rpy="0 0 0" />
@@ -254,6 +254,6 @@
   </link>
   <joint name="left_front_wheel_link_joint" type="continuous">
-    <parent link="left_front_steer_hinge_link" />
-    <child link="left_front_wheel_link" />
+    <parent link="$(arg robot_name)/left_front_steer_hinge_link" />
+    <child link="$(arg robot_name)/left_front_wheel_link" />
     <origin xyz="0 0.025 0" rpy="0 0 0" />
     <axis xyz="0 1 0" />
@@ -261,5 +261,5 @@
   </joint>
   <xacro:wheel_transmission name="left_front_wheel_link" />
-  <link name="camera">
+  <link name="$(arg robot_name)/camera">
     <inertial>
       <origin xyz="0 0 0" rpy="0 0 0" />
@@ -278,10 +278,10 @@
   </link>
   <joint name="camera_joint" type="fixed">
-    <parent link="base_link" />
-    <child link="camera" />
+    <parent link="$(arg robot_name)/base_link" />
+    <child link="$(arg robot_name)/camera" />
     <origin xyz="0.077 0 0.046" rpy="0 0 0" />
     <axis xyz="0 0 0" />
   </joint>
-  <link name="lidar_2d">
+  <link name="$(arg robot_name)/lidar_2d">
     <inertial>
       <origin xyz="0 0 0" rpy="0 0 0" />
@@ -301,9 +301,9 @@
   <joint name="laser_joint" type="fixed">
     <origin xyz="-0.02 0 0.12" rpy="0 0 0" />
-    <parent link="base_link" />
-    <child link="lidar_2d" />
+    <parent link="$(arg robot_name)/base_link" />
+    <child link="$(arg robot_name)/lidar_2d" />
     <axis xyz="0 0 0" />
   </joint>
-  <link name="imu">
+  <link name="$(arg robot_name)/imu">
     <visual>
       <geometry>
@@ -317,6 +317,6 @@
   </link>
   <joint name="imu_joint" type="fixed">
-    <parent link="base_link" />
-    <child link="imu" />
+    <parent link="$(arg robot_name)/base_link" />
+    <child link="$(arg robot_name)/imu" />
     <origin xyz="-0.10 0 0.01" />
     <axis xyz="0 0 1" />

Commit message: tune pid

File: robot_gazebo/urdf/pav_s01/pav_s01.xacro (robot description, xacro)
@@ -157,5 +157,5 @@
     <child link="$(arg robot_name)/left_front_steer_hinge_link" />
     <axis xyz="0 0 1" />
-    <limit lower="-0.6" upper="0.6" effort="5" velocity="1000" />
+    <limit lower="-0.5" upper="0.5" effort="5" velocity="1000" />
   </joint>
   <xacro:steering_hinge_transmission name="left_front_steer_hinge_link" />
@@ -197,5 +197,5 @@
     <origin xyz="0.095 -0.065 -0.0525" rpy="0 0 0" />
     <axis xyz="0 0 1" />
-    <limit lower="-0.6" upper="0.6" effort="5" velocity="1000" />
+    <limit lower="-0.5" upper="0.5" effort="5" velocity="1000" />
   </joint>
   <xacro:steering_hinge_transmission name="right_front_steer_hinge_link" />
