Commit message: tuned pavs00

File: robot_gazebo/urdf/pav_s00/macros.xacro (robot description, xacro)
@@ -1,28 +1,39 @@
 <?xml version="1.0"?>
-<robot name="$(arg robot_name)" xmlns:xacro="http://www.ros.org/wiki/xacro">
-<!-- transmission macros -->
-<xacro:macro name="wheel_transmission" params="name">
-  <transmission name="${name}_transmission" type="SimpleTransmission">
-    <type>transmission_interface/SimpleTransmission</type>
-    <joint name="${name}_joint">
-      <hardwareInterface>hardware_interface/EffortJointInterface</hardwareInterface>
-    </joint>
-    <actuator name="${name}_motor">
-      <hardwareInterface>hardware_interface/EffortJointInterface</hardwareInterface>
-      <mechanicalReduction>1</mechanicalReduction>
-    </actuator>
-  </transmission>
-</xacro:macro>
-<xacro:macro name="steering_hinge_transmission" params="name">
-  <transmission name="${name}_transmission" type="SimpleTransmission">
-    <type>transmission_interface/SimpleTransmission</type>
-    <joint name="${name}_joint">
-      <hardwareInterface>hardware_interface/EffortJointInterface</hardwareInterface>
-    </joint>
-    <actuator name="${name}_motor">
-      <hardwareInterface>hardware_interface/EffortJointInterface</hardwareInterface>
-      <mechanicalReduction>1</mechanicalReduction>
-    </actuator>
-  </transmission>
-</xacro:macro>
+<robot name="$(arg robot_name)"
+  xmlns:xacro="http://www.ros.org/wiki/xacro">
+  <!-- transmission macros -->
+  <xacro:macro name="wheel_transmission" params="name">
+    <transmission name="${name}_transmission" type="SimpleTransmission">
+      <type>transmission_interface/SimpleTransmission</type>
+      <joint name="${name}_joint">
+        <hardwareInterface>hardware_interface/EffortJointInterface</hardwareInterface>
+      </joint>
+      <actuator name="${name}_motor">
+        <hardwareInterface>hardware_interface/EffortJointInterface</hardwareInterface>
+        <mechanicalReduction>1</mechanicalReduction>
+      </actuator>
+    </transmission>
+  </xacro:macro>
+  <xacro:macro name="steering_hinge_transmission" params="name">
+    <transmission name="${name}_transmission" type="SimpleTransmission">
+      <type>transmission_interface/SimpleTransmission</type>
+      <joint name="${name}_joint">
+        <hardwareInterface>hardware_interface/EffortJointInterface</hardwareInterface>
+      </joint>
+      <actuator name="${name}_motor">
+        <hardwareInterface>hardware_interface/EffortJointInterface</hardwareInterface>
+        <mechanicalReduction>1</mechanicalReduction>
+      </actuator>
+    </transmission>
+  </xacro:macro>
+  <xacro:macro name="wheel_friction" params="name">
+    <surface>
+      <friction>
+        <ode>
+          <mu>999999999999999999</mu>
+          <mu2>999999999999999999</mu2>
+        </ode>
+      </friction>
+    </surface>
+  </xacro:macro>
 </robot>

File: robot_gazebo/urdf/pav_s00/pav_s00.xacro (robot description, xacro)
@@ -2,7 +2,10 @@
 <robot name="$(arg robot_name)"
   xmlns:xacro="http://ros.org/wiki/xacro">
+  <xacro:property name="M_PI" value="3.141592653589793" />
+  <xacro:property name="rotation_fiction" value="1"/>
+  <xacro:property name="mu" value="9999999999.0"/>
   <xacro:include filename="$(find robot_gazebo)/urdf/pav_s00/macros.xacro" />
-  <link name="base_footprint"/>
-  <link name="base_link">
+  <link name="$(arg robot_name)/base_footprint"/>
+  <link name="$(arg robot_name)/base_link">
     <inertial>
       <origin xyz="-0.02 0 0" rpy="0 0 0" />
@@ -13,5 +16,5 @@
       <origin xyz="-0.024 0 -0.067" rpy="0 0 0" />
       <geometry>
-        <mesh filename="package://robot_gazebo/models/robots/pav_s00/base_link.STL" />
+        <mesh filename="package://robot_gazebo/models/robots/pav_s01/base_link.STL" />
       </geometry>
       <!-- <origin xyz="-0.02 0 -0.0325" rpy="0 0 0" />
@@ -31,11 +34,11 @@
   </link>
   <joint name="base_joint" type="fixed">
-    <parent link="base_footprint"/>
-    <child link="base_link"/>
+    <parent link="$(arg robot_name)/base_footprint"/>
+    <child link="$(arg robot_name)/base_link"/>
     <origin xyz="0.0 0.0 0.09" rpy="0 0 0"/>
   </joint>
-  <link name="shell_link">
-    <visual>
-      <origin xyz="0 0 0" rpy="1.57 0 -1.57" />
+  <link name="$(arg robot_name)/shell_link">
+    <visual>
+      <origin xyz="0 0 0" rpy="${M_PI/2} 0 -${M_PI/2}" />
       <geometry>
         <mesh filename="package://robot_gazebo/models/robots/pav_s00/shell_pav_s00.STL" scale="0.001 0.001 0.001"/>
@@ -44,9 +47,9 @@
   </link>
   <joint name="shell_link_joint" type="fixed">
-    <parent link="base_link"/>
-    <child link="shell_link"/>
-    <origin xyz="-0.02 0.0 -0.082" rpy="0 0 0"/>
-  </joint>
-  <link name="right_rear_wheel_link">
+    <parent link="$(arg robot_name)/base_link"/>
+    <child link="$(arg robot_name)/shell_link"/>
+    <origin xyz="-0.02 0.0 -0.085" rpy="0 0 0"/>
+  </joint>
+  <link name="$(arg robot_name)/right_rear_wheel_link">
     <inertial>
       <origin xyz="0 0 0 " rpy="0 0 0" />
@@ -59,5 +62,5 @@
         <mesh filename="package://robot_gazebo/models/robots/pav_s00/wheel_link.STL" />
       </geometry>
-      <!-- <origin xyz="0 0 0" rpy="1.57 0 0" />
+      <!-- <origin xyz="0 0 0" rpy="${M_PI/2} 0 0" />
       <geometry>
         <cylinder radius="0.035" length="0.02" />
@@ -68,13 +71,14 @@
     </visual>
     <collision>
-      <origin xyz="0 0 0" rpy="1.57 0 0" />
-      <geometry>
-        <cylinder radius="0.035" length="0.02" />
-      </geometry>
-    </collision>
+      <origin xyz="0 0 0" rpy="${M_PI/2} 0 0" />
+      <geometry>
+        <cylinder radius="0.035" length="0.02" />
+      </geometry>
+    </collision>
+    <xacro:wheel_friction name="${mu}" />
   </link>
   <joint name="right_rear_wheel_link_joint" type="continuous">
-    <parent link="base_link" />
-    <child link="right_rear_wheel_link" />
+    <parent link="$(arg robot_name)/base_link" />
+    <child link="$(arg robot_name)/right_rear_wheel_link" />
     <origin xyz="-0.139 -0.09 -0.055" rpy="0 0 0" />
     <axis xyz="0 1 0" />
@@ -82,16 +86,16 @@
   </joint>
   <xacro:wheel_transmission name="right_rear_wheel_link" />
-  <link name="left_rear_wheel_link">
+  <link name="$(arg robot_name)/left_rear_wheel_link">
     <inertial>
       <origin xyz="0 0 0 " rpy="0 0 0" />
       <mass value="2" />
-     <inertia ixx="6.79E-04" ixy="0" ixz="0" iyy="6.79E-04" iyz="0" izz="1.25E-03" />
-    </inertial>
-    <visual>
-      <origin xyz="0 0 0" rpy="0 0 3.14" />
+      <inertia ixx="6.79E-04" ixy="0" ixz="0" iyy="6.79E-04" iyz="0" izz="1.25E-03" />
+    </inertial>
+    <visual>
+      <origin xyz="0 0 0" rpy="0 0 ${M_PI}" />
       <geometry>
         <mesh filename="package://robot_gazebo/models/robots/pav_s00/wheel_link.STL" />
       </geometry>
-      <!-- <origin xyz="0 0 0" rpy="1.57 0 0" />
+      <!-- <origin xyz="0 0 0" rpy="${M_PI/2} 0 0" />
       <geometry>
         <cylinder radius="0.035" length="0.02" />
@@ -102,19 +106,21 @@
     </visual>
     <collision>
-      <origin xyz="0 0 0" rpy="1.57 0 0" />
-      <geometry>
-        <cylinder radius="0.035" length="0.02" />
-      </geometry>
-    </collision>
+      <origin xyz="0 0 0" rpy="${M_PI/2} 0 0" />
+      <geometry>
+        <cylinder radius="0.035" length="0.02" />
+      </geometry>
+    </collision>
+    <xacro:wheel_friction name="${mu}" />
   </link>
   <joint name="left_rear_wheel_link_joint" type="continuous">
-    <parent link="base_link" />
-    <child link="left_rear_wheel_link" />
+    <parent link="$(arg robot_name)/base_link" />
+    <child link="$(arg robot_name)/left_rear_wheel_link" />
     <origin xyz="-0.139 0.09 -0.055" rpy="0 0 0" />
     <axis xyz="0 1 0" />
     <limit effort="10" velocity="1000" />
+    <dynamics damping="0.0" friction="${rotation_fiction}"/>
   </joint>
   <xacro:wheel_transmission name="left_rear_wheel_link" />
-  <link name="left_front_steer_hinge_link">
+  <link name="$(arg robot_name)/left_front_steer_hinge_link">
     <inertial>
       <origin xyz="0 0 0" rpy="0 0 0" />
@@ -127,5 +133,5 @@
         <mesh filename="package://robot_gazebo/models/robots/pav_s00/steer_hinge_link.STL" />
       </geometry>
-      <!-- <origin xyz="0.0 0.0 0.0" rpy="1.57 0.0 0.0" />
+      <!-- <origin xyz="0.0 0.0 0.0" rpy="${M_PI/2} 0.0 0.0" />
       <geometry>
           <cylinder radius="0.01" length="0.005" />
@@ -141,18 +147,18 @@
       </geometry> -->
       <geometry>
-          <cylinder radius="0.01" length="0.005" />
-      </geometry>
-      <origin xyz="0.0 0.0 0.0" rpy="1.57 0.0 0.0" />
+        <cylinder radius="0.01" length="0.005" />
+      </geometry>
+      <origin xyz="0.0 0.0 0.0" rpy="${M_PI/2} 0.0 0.0" />
     </collision>
   </link>
   <joint name="left_front_steer_hinge_link_joint" type="revolute">
     <origin xyz="0.095 0.065 -0.0525" rpy="0 0 0" />
-    <parent link="base_link" />
-    <child link="left_front_steer_hinge_link" />
+    <parent link="$(arg robot_name)/base_link" />
+    <child link="$(arg robot_name)/left_front_steer_hinge_link" />
     <axis xyz="0 0 1" />
-    <limit lower="-0.6" upper="0.6" effort="5" velocity="1000" />
+    <limit lower="-0.5" upper="0.5" effort="5" velocity="1000" />
   </joint>
   <xacro:steering_hinge_transmission name="left_front_steer_hinge_link" />
-  <link name="right_front_steer_hinge_link">
+  <link name="$(arg robot_name)/right_front_steer_hinge_link">
     <inertial>
       <origin xyz="0 0 0" rpy="0 0 0" />
@@ -165,5 +171,5 @@
         <mesh filename="package://robot_gazebo/models/robots/pav_s00/steer_hinge_link.STL" />
       </geometry>
-      <!-- <origin xyz="0.0 0.0 0.0" rpy="1.57 0.0 0.0" />
+      <!-- <origin xyz="0.0 0.0 0.0" rpy="${M_PI/2} 0.0 0.0" />
       <geometry>
           <cylinder radius="0.01" length="0.005" />
@@ -179,20 +185,20 @@
       </geometry>
     </collision> -->
-      <collision>
-        <geometry>
-            <cylinder radius="0.01" length="0.005" />
-        </geometry>
-        <origin xyz="0.0 0.0 0.0" rpy="1.57 0.0 0.0" />
-      </collision>
+    <collision>
+      <geometry>
+        <cylinder radius="0.01" length="0.005" />
+      </geometry>
+      <origin xyz="0.0 0.0 0.0" rpy="${M_PI/2} 0.0 0.0" />
+    </collision>
   </link>
   <joint name="right_front_steer_hinge_link_joint" type="revolute">
-    <parent link="base_link" />
-    <child link="right_front_steer_hinge_link" />
+    <parent link="$(arg robot_name)/base_link" />
+    <child link="$(arg robot_name)/right_front_steer_hinge_link" />
     <origin xyz="0.095 -0.065 -0.0525" rpy="0 0 0" />
     <axis xyz="0 0 1" />
-    <limit lower="-0.6" upper="0.6" effort="5" velocity="1000" />
+    <limit lower="-0.5" upper="0.5" effort="5" velocity="1000" />
   </joint>
   <xacro:steering_hinge_transmission name="right_front_steer_hinge_link" />
-  <link name="right_front_wheel_link">
+  <link name="$(arg robot_name)/right_front_wheel_link">
     <inertial>
       <origin xyz="0 0 0 " rpy="0 0 0" />
@@ -205,5 +211,5 @@
         <mesh filename="package://robot_gazebo/models/robots/pav_s00/wheel_link.STL" />
       </geometry>
-      <!-- <origin xyz="0 0 0" rpy="1.57 0 0" />
+      <!-- <origin xyz="0 0 0" rpy="${M_PI/2} 0 0" />
       <geometry>
         <cylinder radius="0.035" length="0.02" />
@@ -214,19 +220,21 @@
     </visual>
     <collision>
-      <origin xyz="0 0 0" rpy="1.57 0 0" />
-      <geometry>
-        <cylinder radius="0.035" length="0.02" />
-      </geometry>
-    </collision>
+      <origin xyz="0 0 0" rpy="${M_PI/2} 0 0" />
+      <geometry>
+        <cylinder radius="0.035" length="0.02" />
+      </geometry>
+    </collision>
+    <xacro:wheel_friction name="${mu}" />
   </link>
   <joint name="right_front_wheel_link_joint" type="continuous">
-    <parent link="right_front_steer_hinge_link" />
-    <child link="right_front_wheel_link" />
+    <parent link="$(arg robot_name)/right_front_steer_hinge_link" />
+    <child link="$(arg robot_name)/right_front_wheel_link" />
     <origin xyz="0 -0.025 0" rpy="0 0 0" />
     <axis xyz="0 1 0" />
     <limit effort="10" velocity="1000" />
+    <dynamics damping="0.0" friction="${rotation_fiction}"/>
   </joint>
   <xacro:wheel_transmission name="right_front_wheel_link" />
-  <link name="left_front_wheel_link">
+  <link name="$(arg robot_name)/left_front_wheel_link">
     <inertial>
       <origin xyz="0 0 0 " rpy="0 0 0" />
@@ -235,9 +243,9 @@
     </inertial>
     <visual>
-      <origin xyz="0 0 0" rpy="0 0 3.14" />
+      <origin xyz="0 0 0" rpy="0 0 ${M_PI}" />
       <geometry>
         <mesh filename="package://robot_gazebo/models/robots/pav_s00/wheel_link.STL" />
       </geometry>
-      <!-- <origin xyz="0 0 0" rpy="1.57 0 0" />
+      <!-- <origin xyz="0 0 0" rpy="${M_PI/2} 0 0" />
       <geometry>
         <cylinder radius="0.035" length="0.02" />
@@ -248,19 +256,21 @@
     </visual>
     <collision>
-      <origin xyz="0 0 0" rpy="1.57 0 0" />
-      <geometry>
-        <cylinder radius="0.035" length="0.02" />
-      </geometry>
-    </collision>
+      <origin xyz="0 0 0" rpy="${M_PI/2} 0 0" />
+      <geometry>
+        <cylinder radius="0.035" length="0.02" />
+      </geometry>
+    </collision>
+    <xacro:wheel_friction name="${mu}" />
   </link>
   <joint name="left_front_wheel_link_joint" type="continuous">
-    <parent link="left_front_steer_hinge_link" />
-    <child link="left_front_wheel_link" />
+    <parent link="$(arg robot_name)/left_front_steer_hinge_link" />
+    <child link="$(arg robot_name)/left_front_wheel_link" />
     <origin xyz="0 0.025 0" rpy="0 0 0" />
     <axis xyz="0 1 0" />
     <limit effort="10" velocity="1000" />
+    <dynamics damping="0.0" friction="${rotation_fiction}"/>
   </joint>
   <xacro:wheel_transmission name="left_front_wheel_link" />
-  <link name="camera">
+  <link name="$(arg robot_name)/camera">
     <inertial>
       <origin xyz="0 0 0" rpy="0 0 0" />
@@ -279,7 +289,14 @@
   </link>
   <joint name="camera_joint" type="fixed">
-    <parent link="base_link" />
-    <child link="camera" />
+    <parent link="$(arg robot_name)/base_link" />
+    <child link="$(arg robot_name)/camera" />
     <origin xyz="0.077 0 0.046" rpy="0 0 0" />
+    <axis xyz="0 0 0" />
+  </joint>
+  <link name="$(arg robot_name)/depth_camera"/>
+  <joint name="depth_camera_joint" type="fixed">
+    <parent link="$(arg robot_name)/camera" />
+    <child link="$(arg robot_name)/depth_camera" />
+    <origin xyz="0 0 0" rpy="-${M_PI/2} 0 -${M_PI/2}" />
     <axis xyz="0 0 0" />
   </joint>
@@ -287,8 +304,8 @@
   <xacro:property name="gpu" value="$(arg gpu)" />
   <xacro:include filename="$(find robot_gazebo)/urdf/pav_s00/pav_s00_VLP-16.urdf.xacro"/>
-  <xacro:VLP-16 parent="base_link" name="velodyne" topic="/velodyne_points" hz="10" samples="440" gpu="${gpu}">
+  <xacro:VLP-16 parent="$(arg robot_name)/base_link" name="$(arg robot_name)/velodyne" topic="/velodyne_points" hz="10" samples="440" gpu="${gpu}">
     <origin xyz="-0.022 0 0.1" rpy="0 0 0" />
   </xacro:VLP-16>
-  <link name="imu">
+  <link name="$(arg robot_name)/imu">
     <visual>
       <geometry>
@@ -302,6 +319,6 @@
   </link>
   <joint name="imu_joint" type="fixed">
-    <parent link="base_link" />
-    <child link="imu" />
+    <parent link="$(arg robot_name)/base_link" />
+    <child link="$(arg robot_name)/imu" />
     <origin xyz="-0.10 0 0.01" />
     <axis xyz="0 0 1" />

File: robot_gazebo/urdf/pav_s00/pav_s00_VLP-16.urdf.xacro (robot description, xacro)
@@ -3,9 +3,4 @@
   <xacro:property name="M_PI" value="3.1415926535897931" />
   <xacro:macro name="VLP-16" params="*origin parent:=base_link name:=velodyne topic:=/velodyne_points hz:=10 lasers:=16 samples:=1875 collision_range:=0.3 min_range:=0.9 max_range:=130.0 noise:=0.008 min_angle:=-${M_PI} max_angle:=${M_PI} gpu:=false">
-    <joint name="${name}_base_mount_joint" type="fixed">
-      <xacro:insert_block name="origin" />
-      <parent link="${parent}"/>
-      <child link="${name}_base_link"/>
-    </joint>
     <link name="${name}_base_link">
       <visual>
@@ -26,4 +21,9 @@
       </collision>
     </link>
+    <joint name="${name}_base_mount_joint" type="fixed">
+      <xacro:insert_block name="origin" />
+      <parent link="${parent}"/>
+      <child link="${name}_base_link"/>
+    </joint>
     <joint name="${name}_base_scan_joint" type="fixed" >
       <origin xyz="0 0 0.0377" rpy="0 0 0" />
@@ -74,5 +74,5 @@
           <plugin name="gazebo_ros_laser_controller" filename="libgazebo_ros_velodyne_gpu_laser.so">
             <topicName>${topic}</topicName>
-            <frameName>${name}</frameName>
+            <frameName>velodyne</frameName>
             <min_range>${min_range}</min_range>
             <max_range>${max_range}</max_range>
@@ -114,5 +114,5 @@
           <plugin name="gazebo_ros_laser_controller" filename="libgazebo_ros_velodyne_laser.so">
             <topicName>${topic}</topicName>
-            <frameName>${name}</frameName>
+            <frameName>velodyne</frameName>
             <min_range>${min_range}</min_range>
             <max_range>${max_range}</max_range>

File: robot_gazebo/urdf/pav_s01/macros.xacro (robot description, xacro)
@@ -1,38 +1,39 @@
 <?xml version="1.0"?>
-<robot name="$(arg robot_name)" xmlns:xacro="http://ros.org/wiki/xacro">
-<!-- transmission macros -->
-<xacro:macro name="wheel_transmission" params="name">
-  <transmission name="${name}_transmission" type="SimpleTransmission">
-    <type>transmission_interface/SimpleTransmission</type>
-    <joint name="${name}_joint">
-      <hardwareInterface>hardware_interface/EffortJointInterface</hardwareInterface>
-    </joint>
-    <actuator name="${name}_motor">
-      <hardwareInterface>hardware_interface/EffortJointInterface</hardwareInterface>
-      <mechanicalReduction>1</mechanicalReduction>
-    </actuator>
-  </transmission>
-</xacro:macro>
-<xacro:macro name="steering_hinge_transmission" params="name">
-  <transmission name="${name}_transmission" type="SimpleTransmission">
-    <type>transmission_interface/SimpleTransmission</type>
-    <joint name="${name}_joint">
-      <hardwareInterface>hardware_interface/EffortJointInterface</hardwareInterface>
-    </joint>
-    <actuator name="${name}_motor">
-      <hardwareInterface>hardware_interface/EffortJointInterface</hardwareInterface>
-      <mechanicalReduction>1</mechanicalReduction>
-    </actuator>
-  </transmission>
-</xacro:macro>
-<xacro:macro name="wheel_friction" params="name">
-  <surface>
+<robot name="$(arg robot_name)"
+  xmlns:xacro="http://ros.org/wiki/xacro">
+  <!-- transmission macros -->
+  <xacro:macro name="wheel_transmission" params="name">
+    <transmission name="${name}_transmission" type="SimpleTransmission">
+      <type>transmission_interface/SimpleTransmission</type>
+      <joint name="${name}_joint">
+        <hardwareInterface>hardware_interface/EffortJointInterface</hardwareInterface>
+      </joint>
+      <actuator name="${name}_motor">
+        <hardwareInterface>hardware_interface/EffortJointInterface</hardwareInterface>
+        <mechanicalReduction>1</mechanicalReduction>
+      </actuator>
+    </transmission>
+  </xacro:macro>
+  <xacro:macro name="steering_hinge_transmission" params="name">
+    <transmission name="${name}_transmission" type="SimpleTransmission">
+      <type>transmission_interface/SimpleTransmission</type>
+      <joint name="${name}_joint">
+        <hardwareInterface>hardware_interface/EffortJointInterface</hardwareInterface>
+      </joint>
+      <actuator name="${name}_motor">
+        <hardwareInterface>hardware_interface/EffortJointInterface</hardwareInterface>
+        <mechanicalReduction>1</mechanicalReduction>
+      </actuator>
+    </transmission>
+  </xacro:macro>
+  <xacro:macro name="wheel_friction" params="name">
+    <surface>
       <friction>
         <ode>
-            <mu>999999999999999999</mu>
-            <mu2>999999999999999999</mu2>
+          <mu>999999999999999999</mu>
+          <mu2>999999999999999999</mu2>
         </ode>
       </friction>
-  </surface>
-</xacro:macro>
+    </surface>
+  </xacro:macro>
 </robot>

File: robot_gazebo/urdf/pav_s01/pav_s01.xacro (robot description, xacro)
@@ -1,4 +1,5 @@
 <?xml version="1.0" encoding="utf-8"?>
-<robot name="$(arg robot_name)" xmlns:xacro="http://ros.org/wiki/xacro">
+<robot name="$(arg robot_name)"
+  xmlns:xacro="http://ros.org/wiki/xacro">
   <xacro:property name="M_PI" value="3.141592653589793" />
   <xacro:property name="rotation_fiction" value="1"/>
@@ -90,5 +91,5 @@
       <origin xyz="0 0 0 " rpy="0 0 0" />
       <mass value="2" />
-     <inertia ixx="6.79E-04" ixy="0" ixz="0" iyy="6.79E-04" iyz="0" izz="1.25E-03" />
+      <inertia ixx="6.79E-04" ixy="0" ixz="0" iyy="6.79E-04" iyz="0" izz="1.25E-03" />
     </inertial>
     <visual>
@@ -147,5 +148,5 @@
       </geometry> -->
       <geometry>
-          <cylinder radius="0.01" length="0.005" />
+        <cylinder radius="0.01" length="0.005" />
       </geometry>
       <origin xyz="0.0 0.0 0.0" rpy="${M_PI/2} 0.0 0.0" />
@@ -185,10 +186,10 @@
       </geometry>
     </collision> -->
-      <collision>
-        <geometry>
-            <cylinder radius="0.01" length="0.005" />
-        </geometry>
-        <origin xyz="0.0 0.0 0.0" rpy="${M_PI/2} 0.0 0.0" />
-      </collision>
+    <collision>
+      <geometry>
+        <cylinder radius="0.01" length="0.005" />
+      </geometry>
+      <origin xyz="0.0 0.0 0.0" rpy="${M_PI/2} 0.0 0.0" />
+    </collision>
   </link>
   <joint name="right_front_steer_hinge_link_joint" type="revolute">
